File: board/hdmilight.sch (EAGLE design)
At the start: 73 parts, among them IC1 REG1117, IC2 REG1117, J1 POWER_JACKPTH, Q1 28.6363MHz

Commit message: fixed value of HDMI pull up resistors on receiver board
Parts:
- R1: value 27R -> 27K
- R2, R3: value 47R -> 1K5
- R7, R8: value 47R -> 47K
- R9: value 100R -> 100K
Changed lines of the file:
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@@
 <part name="C1" library="resistor" deviceset="C-EU" device="C0603" value="0.1uF"/>
 <part name="GND12" library="supply1" deviceset="GND" device=""/>
-<part name="R2" library="resistor" deviceset="R-EU_" device="R0603" value="47R"/>
-<part name="R3" library="resistor" deviceset="R-EU_" device="R0603" value="47R"/>
-<part name="R7" library="resistor" deviceset="R-EU_" device="R0603" value="47R"/>
-<part name="R8" library="resistor" deviceset="R-EU_" device="R0603" value="47R"/>
+<part name="R2" library="resistor" deviceset="R-EU_" device="R0603" value="1K5"/>
+<part name="R3" library="resistor" deviceset="R-EU_" device="R0603" value="1K5"/>
+<part name="R7" library="resistor" deviceset="R-EU_" device="R0603" value="47K"/>
+<part name="R8" library="resistor" deviceset="R-EU_" device="R0603" value="47K"/>
 <part name="SUPPLY12" library="supply2" deviceset="V&lt;--" device="" value="VCC_3V3"/>
-<part name="R1" library="resistor" deviceset="R-EU_" device="R0603" value="27R"/>
-<part name="R9" library="resistor" deviceset="R-EU_" device="R0603" value="100R"/>
+<part name="R1" library="resistor" deviceset="R-EU_" device="R0603" value="27K"/>
+<part name="R9" library="resistor" deviceset="R-EU_" device="R0603" value="100K"/>
 <part name="SUPPLY13" library="supply2" deviceset="V&lt;--" device="" value="VCC_3V3"/>
 <part name="GND13" library="supply1" deviceset="GND" device=""/>

Commit message: added missing capacitor values to schematic
Parts:
- C15, C16, C17, C18, C19, C20, C21, C22, C23, C24, C25, C26, C33, C34, C35, C36, C37: value (none) -> 0.1uF
Changed lines of the file:
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@@
 <part name="GND15" library="supply1" deviceset="GND" device=""/>
 <part name="GND16" library="supply1" deviceset="GND" device=""/>
-<part name="C22" library="resistor" deviceset="C-EU" device="C0603"/>
-<part name="C15" library="resistor" deviceset="C-EU" device="C0402"/>
-<part name="C23" library="resistor" deviceset="C-EU" device="C0402"/>
-<part name="C34" library="resistor" deviceset="C-EU" device="C0402"/>
-<part name="C16" library="resistor" deviceset="C-EU" device="C0603"/>
-<part name="C17" library="resistor" deviceset="C-EU" device="C0603"/>
-<part name="C24" library="resistor" deviceset="C-EU" device="C0603"/>
-<part name="C35" library="resistor" deviceset="C-EU" device="C0603"/>
-<part name="C18" library="resistor" deviceset="C-EU" device="C0402"/>
-<part name="C19" library="resistor" deviceset="C-EU" device="C0603"/>
+<part name="C22" library="resistor" deviceset="C-EU" device="C0603" value="0.1uF"/>
+<part name="C15" library="resistor" deviceset="C-EU" device="C0402" value="0.1uF"/>
+<part name="C23" library="resistor" deviceset="C-EU" device="C0402" value="0.1uF"/>
+<part name="C34" library="resistor" deviceset="C-EU" device="C0402" value="0.1uF"/>
+<part name="C16" library="resistor" deviceset="C-EU" device="C0603" value="0.1uF"/>
+<part name="C17" library="resistor" deviceset="C-EU" device="C0603" value="0.1uF"/>
+<part name="C24" library="resistor" deviceset="C-EU" device="C0603" value="0.1uF"/>
+<part name="C35" library="resistor" deviceset="C-EU" device="C0603" value="0.1uF"/>
+<part name="C18" library="resistor" deviceset="C-EU" device="C0402" value="0.1uF"/>
+<part name="C19" library="resistor" deviceset="C-EU" device="C0603" value="0.1uF"/>
 <part name="GND10" library="supply1" deviceset="GND" device=""/>
 <part name="GND17" library="supply1" deviceset="GND" device=""/>
@@
 <part name="SUPPLY17" library="supply2" deviceset="V&lt;--" device="" value="TVDD_3V3"/>
 <part name="SUPPLY18" library="supply2" deviceset="V&lt;--" device="" value="VCC_3V3"/>
-<part name="C37" library="resistor" deviceset="C-EU" device="C0402"/>
-<part name="C33" library="resistor" deviceset="C-EU" device="C0603"/>
-<part name="C25" library="resistor" deviceset="C-EU" device="C0402"/>
-<part name="C36" library="resistor" deviceset="C-EU" device="C0402"/>
+<part name="C37" library="resistor" deviceset="C-EU" device="C0402" value="0.1uF"/>
+<part name="C33" library="resistor" deviceset="C-EU" device="C0603" value="0.1uF"/>
+<part name="C25" library="resistor" deviceset="C-EU" device="C0402" value="0.1uF"/>
+<part name="C36" library="resistor" deviceset="C-EU" device="C0402" value="0.1uF"/>
 <part name="GND22" library="supply1" deviceset="GND" device=""/>
 <part name="R6" library="resistor" deviceset="R-EU_" device="R0603" value="1K"/>
@@
 <part name="SUPPLY20" library="supply2" deviceset="V&lt;--" device="" value="VCC_5V0"/>
 <part name="SUPPLY21" library="supply2" deviceset="V&lt;--" device="" value="VCC_5V0"/>
-<part name="C20" library="resistor" deviceset="C-EU" device="C0603"/>
+<part name="C20" library="resistor" deviceset="C-EU" device="C0603" value="0.1uF"/>
 <part name="+3V3" library="supply1" deviceset="+3V3" device=""/>
 <part name="GND27" library="supply1" deviceset="GND" device=""/>
 <part name="SUPPLY22" library="supply2" deviceset="V&lt;--" device="" value="VCC_5V0"/>
-<part name="C21" library="resistor" deviceset="C-EU" device="C0603"/>
-<part name="C26" library="resistor" deviceset="C-EU" device="C0603"/>
+<part name="C21" library="resistor" deviceset="C-EU" device="C0603" value="0.1uF"/>
+<part name="C26" library="resistor" deviceset="C-EU" device="C0603" value="0.1uF"/>
 <part name="GND28" library="supply1" deviceset="GND" device=""/>
 <part name="R13" library="resistor" deviceset="R-EU_" device="R0603" value="4K7"/>

Commit message: removed power jack from HDMI receiver board
Parts:
- removed J1: POWER_JACKPTH, SparkFun:POWER_JACKPTH
Connections:
- removed net N$17: F1.1, J1.PWR, R11.1
- net +5V: now also F1.1, R11.1; no longer J1.GNDBREAK
- net GND: no longer J1.GND
Changed lines of the file:
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@@
 <part name="C8" library="resistor" deviceset="C-EU" device="C1206" value="22uF"/>
 <part name="GND2" library="supply1" deviceset="GND" device=""/>
-<part name="J1" library="SparkFun" deviceset="POWER_JACK" device="PTH"/>
 <part name="GND3" library="supply1" deviceset="GND" device=""/>
 <part name="SV1" library="con-lstb" deviceset="MA08-2" device=""/>
@@
 <instance part="C8" gate="G$1" x="304.8" y="116.84"/>
 <instance part="GND2" gate="1" x="287.02" y="101.6"/>
-<instance part="J1" gate="G$1" x="187.96" y="185.42"/>
 <instance part="GND3" gate="1" x="220.98" y="160.02"/>
 <instance part="SV1" gate="G$1" x="63.5" y="243.84" rot="MR0"/>
@@
 <instance part="R10" gate="G$1" x="86.36" y="180.34"/>
 <instance part="GND11" gate="1" x="86.36" y="210.82" rot="R180"/>
-<instance part="P+1" gate="1" x="200.66" y="203.2"/>
+<instance part="P+1" gate="1" x="205.74" y="203.2"/>
 <instance part="P+2" gate="1" x="322.58" y="63.5"/>
 <instance part="C1" gate="G$1" x="27.94" y="71.12"/>
@@
 </segment>
 </net>
-<net name="N$17" class="0">
-<segment>
-<wire x1="218.44" y1="193.04" x2="205.74" y2="193.04" width="0.1524" layer="91"/>
-<wire x1="205.74" y1="193.04" x2="205.74" y2="180.34" width="0.1524" layer="91"/>
-<wire x1="190.5" y1="193.04" x2="205.74" y2="193.04" width="0.1524" layer="91"/>
-<junction x="205.74" y="193.04"/>
-<pinref part="F1" gate="G$1" pin="1"/>
-<pinref part="R11" gate="G$1" pin="1"/>
-<pinref part="J1" gate="G$1" pin="PWR"/>
-</segment>
-</net>
 <net name="VCC_5V0" class="0">
 <segment>
@@
 <wire x1="205.74" y1="170.18" x2="205.74" y2="167.64" width="0.1524" layer="91"/>
 <wire x1="205.74" y1="167.64" x2="220.98" y2="167.64" width="0.1524" layer="91"/>
-<wire x1="195.58" y1="167.64" x2="205.74" y2="167.64" width="0.1524" layer="91"/>
-<junction x="205.74" y="167.64"/>
 <junction x="220.98" y="167.64"/>
 <pinref part="C4" gate="G$1" pin="2"/>
 <pinref part="GND3" gate="1" pin="GND"/>
 <pinref part="R11" gate="G$1" pin="2"/>
-<wire x1="190.5" y1="187.96" x2="195.58" y2="187.96" width="0.1524" layer="91"/>
-<pinref part="J1" gate="G$1" pin="GND"/>
-<wire x1="195.58" y1="187.96" x2="195.58" y2="167.64" width="0.1524" layer="91"/>
 </segment>
 <segment>
@@
 <net name="+5V" class="0">
 <segment>
-<pinref part="J1" gate="G$1" pin="GNDBREAK"/>
 <pinref part="P+1" gate="1" pin="+5V"/>
-<wire x1="190.5" y1="190.5" x2="200.66" y2="190.5" width="0.1524" layer="91"/>
-<wire x1="200.66" y1="190.5" x2="200.66" y2="200.66" width="0.1524" layer="91"/>
-</segment>
-<segment>
+<wire x1="218.44" y1="193.04" x2="205.74" y2="193.04" width="0.1524" layer="91"/>
+<wire x1="205.74" y1="193.04" x2="205.74" y2="180.34" width="0.1524" layer="91"/>
+<junction x="205.74" y="193.04"/>
+<pinref part="F1" gate="G$1" pin="1"/>
+<pinref part="R11" gate="G$1" pin="1"/>
+<wire x1="205.74" y1="193.04" x2="205.74" y2="200.66" width="0.1524" layer="91"/>
+</segment>
+<segment>

Commit message: receiver board: replaced TXB0108 level shifter with a 74HCT541
Parts:
- removed C20: 0.1uF, resistor:C-EUC0603
- removed U$5: TXB0108, __SR:TXB0108
- added IC3: 74HCT541DW, 74xx-eu:74HCT541DW
Connections:
- removed net N$46: SV1.10, U$5.B4
- removed net N$47: SV1.8, U$5.B5
- removed net N$48: SV1.6, U$5.B6
- removed net N$49: SV1.4, U$5.B7
- removed net N$50: U$5.A1, U$7C_IO.A9
- removed net N$51: SV1.16, U$5.B1
- new net N$10: IC3A.A7, U$7C_IO.A15
- new net N$11: IC3A.A6, U$7C_IO.A14
- new net N$12: IC3A.A5, U$7C_IO.A13
- new net N$17: IC3A.A4, U$7C_IO.A12
- new net N$42: IC3A.Y3, SV1.12
- new net N$9: IC3A.A8, U$7C_IO.A16
- net +3V3: no longer C20.1, U$5.OE, U$5.VCCA
- net GND: now also IC3A.G1, IC3A.G2, IC3P.GND; no longer C20.2, U$5.GND
- net N$18: now also IC3A.A3, U$7C_IO.A11; no longer SV1.2, U$5.B8
- net N$35: now also IC3A.A2, U$7C_IO.A10; no longer U$5.A8, U$7C_IO.A16
- net N$36: now also IC3A.A1, U$7C_IO.A9; no longer U$5.A7, U$7C_IO.A15
- net N$37: now also IC3A.Y5, SV1.2; no longer U$5.A6, U$7C_IO.A14
- net N$38: now also IC3A.Y8, SV1.8; no longer U$5.A5, U$7C_IO.A13
- net N$39: now also IC3A.Y7, SV1.6; no longer U$5.A4, U$7C_IO.A12
- net N$40: now also IC3A.Y6, SV1.4; no longer U$5.A3, U$7C_IO.A11
- net N$41: now also IC3A.Y4, SV1.10; no longer U$5.A2, U$7C_IO.A10
- net N$44: now also IC3A.Y2; no longer U$5.B2
- net N$45: now also IC3A.Y1, SV1.16; no longer SV1.12, U$5.B3
- net VCC_5V0: now also IC3P.VCC; no longer U$5.VCCB
Other:
- moved on the sheet: C21, C26, SV1

Commit message: receiver board: changed value of IP4776CZ38 ESD protection IC to TPD12S520
Parts:
- U$4: value IP4776CZ38 -> TPD12S520
Changed lines of the file:
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@@
 <part name="U$6" library="__SR" deviceset="ADV7611" device=""/>
 <part name="U$1" library="__SR" deviceset="FCI_HDMI_SOCKET_10029449-001RCF" device=""/>
-<part name="U$4" library="__SR" deviceset="IP4776CZ38" device=""/>
+<part name="U$4" library="__SR" deviceset="IP4776CZ38" device="" value="TPD12S520"/>
 <part name="F1" library="SparkFun" deviceset="PTC" device="SMD" value="1206L050YR"/>
 <part name="R11" library="varistor" deviceset="VARISTOR" device="CN0603" value="V5.5MLA0603H"/>

Commit message: receiver board: merged changes from Jet:
 * added "power" and "hotplug" LED labels
 * added LED polarity symbols
 * moved C7/C8 labels off of vias
 * moved vias from under SCL and RST labels
 * moved vias from under R13/14/15 labels
 * added + symbols on polarised caps C7-14
 * added R16: 10K between VCC_3V3 and TPD12S520 LV_SUPPLY
 * increased drill size for ADV7611 ground pad from 12mil to 13mil
 * fixed schematic net labels

also changed:

 * edited pin header package to remove the "1" and "16" labels
 * added channel number labels to output channel header
 * changed all text to same vector font
 * added OSHW logo
Parts:
- added LOGO1: OSHW_LOGO_FILLX0200-NT, ohw-logo:OSHW_LOGO_FILLX0200-NT
- added R16: 10K, resistor:R-EU_R0603
- C35: device resistor:C-EUC0603 -> resistor:C-EUC0402
Connections:
- new net N$47: C19.1, R16.2, U$4.3V3
- net LLC: now also U$7A_B_IO.A14; no longer U$7A_B_IO.A10
- net P16: now also U$7A_B_IO.A10; no longer U$7A_B_IO.B11
- net P17: now also U$7A_B_IO.B11; no longer U$7A_B_IO.A11
- net P18: now also U$7A_B_IO.A11; no longer U$7A_B_IO.B12
- net P19: now also U$7A_B_IO.B12; no longer U$7A_B_IO.A12
- net P20: now also U$7A_B_IO.A12; no longer U$7A_B_IO.B13
- net P22: now also U$7A_B_IO.A15; no longer U$7A_B_IO.B14
- net P23: now also U$7A_B_IO.A16; no longer U$7A_B_IO.A14
- net VCC_3V3: now also R16.1; no longer C19.1, U$4.3V3
Other:
- moved on the sheet: C19
